File: project-nrf-leak-detector.kicad_sch (KiCad schematic)
At the start: 17 parts, among them J1 Conn_02x05_Odd_Even, J2 Water Probe, Q1 Q_NMOS_GSD, U1 MS88SF3_NRF52840

Commit message: Add missing part numbers
Parts:
- D1: MPN (none) -> CUS10S30,H3F
- Q1: MPN (none) -> RU1J002YNTCL
Changed lines of the file:
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@@
       (effects (font (size 1.27 1.27)) hide)
+    )
+    (property "MPN" "RU1J002YNTCL" (at 157.48 59.69 0)
+      (effects (font (size 1.27 1.27)))
     )
     (pin "1")
@@
       (effects (font (size 1.27 1.27)) hide)
     )
+    (property "MPN" "CUS10S30,H3F" (at 157.48 48.26 90)
+      (effects (font (size 1.27 1.27)))
+    )
     (pin "1")

Commit message: Correct resistor value error
10k -> 1M
Parts:
- R3: value 10k -> 1M
Changed lines of the file:
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@@
     (effects (font (size 1.27 1.27)) (justify left bottom))
   )
-  (label "WATER_PROBE" (at 16.51 68.58 0)
-    (effects (font (size 1.27 1.27)) (justify left bottom))
-  )
-  (label "GND" (at 133.35 110.49 0)
-    (effects (font (size 1.27 1.27)) (justify left bottom))
-  )
-  (label "BUZZER" (at 127 57.15 0)
-    (effects (font (size 1.27 1.27)) (justify left bottom))
-  )
-  (label "BUZZER" (at 16.51 73.66 0)
-    (effects (font (size 1.27 1.27)) (justify left bottom))
-  )
-  (label "SWDIO" (at 21.59 53.34 0)
-    (effects (font (size 1.27 1.27)) (justify left bottom))
-  )
-  (label "SWCLK" (at 21.59 50.8 0)
-    (effects (font (size 1.27 1.27)) (justify left bottom))
-  )
-  (label "~{RESET}" (at 163.83 115.57 180)
+  (label "WATER_PROBE" (at 16.51 68.58 0) (fields_autoplaced)
+    (effects (font (size 1.27 1.27)) (justify left bottom))
+  )
+  (label "GND" (at 133.35 110.49 0) (fields_autoplaced)
+    (effects (font (size 1.27 1.27)) (justify left bottom))
+  )
+  (label "BUZZER" (at 127 57.15 0) (fields_autoplaced)
+    (effects (font (size 1.27 1.27)) (justify left bottom))
+  )
+  (label "BUZZER" (at 16.51 73.66 0) (fields_autoplaced)
+    (effects (font (size 1.27 1.27)) (justify left bottom))
+  )
+  (label "SWDIO" (at 21.59 53.34 0) (fields_autoplaced)
+    (effects (font (size 1.27 1.27)) (justify left bottom))
+  )
+  (label "SWCLK" (at 21.59 50.8 0) (fields_autoplaced)
+    (effects (font (size 1.27 1.27)) (justify left bottom))
+  )
+  (label "~{RESET}" (at 163.83 115.57 180) (fields_autoplaced)
     (effects (font (size 1.27 1.27)) (justify right bottom))
   )
-  (label "RX" (at 100.33 55.88 180)
+  (label "RX" (at 100.33 55.88 180) (fields_autoplaced)
     (effects (font (size 1.27 1.27)) (justify right bottom))
   )
-  (label "~{RESET}" (at 34.29 167.64 0)
-    (effects (font (size 1.27 1.27)) (justify left bottom))
-  )
-  (label "VDD_nRF" (at 133.35 105.41 0)
-    (effects (font (size 1.27 1.27)) (justify left bottom))
-  )
-  (label "RX" (at 163.83 113.03 180)
+  (label "~{RESET}" (at 34.29 167.64 0) (fields_autoplaced)
+    (effects (font (size 1.27 1.27)) (justify left bottom))
+  )
+  (label "VDD_nRF" (at 133.35 105.41 0) (fields_autoplaced)
+    (effects (font (size 1.27 1.27)) (justify left bottom))
+  )
+  (label "RX" (at 163.83 113.03 180) (fields_autoplaced)
     (effects (font (size 1.27 1.27)) (justify right bottom))
   )
-  (label "SWDIO" (at 163.83 105.41 180)
+  (label "SWDIO" (at 163.83 105.41 180) (fields_autoplaced)
     (effects (font (size 1.27 1.27)) (justify right bottom))
   )
-  (label "GND" (at 133.35 107.95 0)
-    (effects (font (size 1.27 1.27)) (justify left bottom))
-  )
-  (label "TX" (at 163.83 110.49 180)
+  (label "GND" (at 133.35 107.95 0) (fields_autoplaced)
+    (effects (font (size 1.27 1.27)) (justify left bottom))
+  )
+  (label "TX" (at 163.83 110.49 180) (fields_autoplaced)
     (effects (font (size 1.27 1.27)) (justify right bottom))
   )
-  (label "WATER_PROBE" (at 237.49 33.02 0)
-    (effects (font (size 1.27 1.27)) (justify left bottom))
-  )
-  (label "SWCLK" (at 163.83 107.95 180)
+  (label "WATER_PROBE" (at 237.49 33.02 0) (fields_autoplaced)
+    (effects (font (size 1.27 1.27)) (justify left bottom))
+  )
+  (label "SWCLK" (at 163.83 107.95 180) (fields_autoplaced)
     (effects (font (size 1.27 1.27)) (justify right bottom))
   )
-  (label "TX" (at 100.33 78.74 180)
+  (label "TX" (at 100.33 78.74 180) (fields_autoplaced)
     (effects (font (size 1.27 1.27)) (justify right bottom))
   )
-  (label "VDD_nRF" (at 101.6 33.02 180)
+  (label "VDD_nRF" (at 101.6 33.02 180) (fields_autoplaced)
     (effects (font (size 1.27 1.27)) (justify right bottom))
   )
-  (label "VDD_nRF" (at 201.93 27.94 180)
+  (label "VDD_nRF" (at 201.93 27.94 180) (fields_autoplaced)
     (effects (font (size 1.27 1.27)) (justify right bottom))
   )
-  (label "~{RESET}" (at 21.59 104.14 0)
-    (effects (font (size 1.27 1.27)) (justify left bottom))
-  )
-  (label "GND" (at 133.35 115.57 0)
+  (label "~{RESET}" (at 21.59 104.14 0) (fields_autoplaced)
+    (effects (font (size 1.27 1.27)) (justify left bottom))
+  )
+  (label "GND" (at 133.35 115.57 0) (fields_autoplaced)
     (effects (font (size 1.27 1.27)) (justify left bottom))
   )
@@
       (effects (font (size 1.27 1.27)) (justify left))
     )
-    (property "Value" "10k" (at 258.318 27.813 0)
-      (effects (font (size 1.27 1.27)) (justify left))
-    )
+    (property "Value" "1M" (at 258.318 27.813 0)
+      (effects (font (size 1.27 1.27)) (justify left))
+    )
